File: Aurora_hardware.sch (KiCad schematic (older format))
At the start: 40 parts

Commit message: avancement carte
Parts:
- removed R2, R? (x25): R, symbol Device:R
- added J: DIGITALOUTNI, symbol Connector:DB9_Female_MountingHoles
- added J: INRELAY, symbol Connector_Generic:Conn_01x11
- added R? (x26): R, symbol Device:R
Connections:
- net labels added: LEDO1-, LEDO2-, LEDO3-, LEDO4-, LEDO5-, LEDO6-, LEDO7-, LEDO8-, LEDO9-, LEDR1-, LEDR2-, LEDR3-, LEDR4-, LEDR5-, LEDR6-, LEDR7-, LEDR8-, LEDR9-, LEDRALIM-, LEDV1-, LEDV2-, LEDV3-, LEDV4-, LEDV5-, LEDV6-, LEDV7-, LEDV8-, LEDV9-, LEDVALIM-, SW1.OUT2, SW2.OUT2, SW3.OUT2, SW4.OUT2, SW5.OUT2, SW6.OUT2, SW7.OUT2, SW8.OUT2, SW9.OUT2, SWALIM.OUT2
- wire segments 95 -> 83
Other:
- moved on the sheet: R1, R?

Commit message: schematic finished
Parts:
- added R11, R17, R22, R27, R32, R37, R42, R47, R5: R, symbol Device:R
- added U1, U2, U3, U4, U5: 4081, symbol 4xxx_IEEE:4081
- gave numbers to parts that had none: 37
- renumbered J to J1, J to J2
Connections:
- net +5V: now also U1.14 (Vdd), U1.14 (Vdd), U1.14 (Vdd), U1.14 (Vdd), U2.14 (Vdd), U2.14 (Vdd), U2.14 (Vdd), U3.14 (Vdd), U3.14 (Vdd), U3.14 (Vdd), U3.14 (Vdd), U4.14 (Vdd), U4.14 (Vdd), U4.14 (Vdd), U5.14 (Vdd), U5.14 (Vdd)
- net GND: now also J2.1 (Pin_1)
- net GNDREF: now also R11.1, R17.1, R22.1, R27.1, R32.1, R37.1, R42.1, R47.1, R5.1, U1.7 (Vss), U1.7 (Vss), U1.7 (Vss), U1.7 (Vss), U2.7 (Vss), U2.7 (Vss), U2.7 (Vss), U2.7 (Vss), U3.7 (Vss), U3.7 (Vss), U3.7 (Vss), U3.7 (Vss), U4.7 (Vss), U4.7 (Vss), U4.7 (Vss), U4.7 (Vss), U5.7 (Vss), U5.7 (Vss)
- net SW1.OUT2: now also U1.1
- net SW2.OUT2: now also U1.5
- net SW3.OUT2: now also U3.5
- net SW4.OUT2: now also U3.8
- net SW5.OUT2: now also U1.8
- net SW6.OUT2: now also U1.12
- net SW7.OUT2: now also U3.12
- net SW8.OUT2: now also U4.1
- net SW9.OUT2: now also U2.1
- net SWALIM.OUT2: now also J2.2 (Pin_2)
- net BP2.OUT2: now reaches JPP2.11, JPP2.12
- net BP2.OUT2: now also R11.2, U2.9
- net BP3.OUT2: now reaches JPP2.16, JPP2.17
- net BP3.OUT2: now also R17.2, U4.9
- net BP4.OUT2: now reaches JPP2.21, JPP2.22
- net BP4.OUT2: now also R22.2, U4.13
- net BP5.OUT2: now reaches JPP2.26, JPP2.27
- net BP5.OUT2: now also R27.2, U2.13
- net BP6.OUT2: now reaches JPP2.31, JPP2.32
- net BP6.OUT2: now also R32.2, U3.2
- net BP7.OUT2: now reaches JPP2.36, JPP2.37
- net BP7.OUT2: now also R37.2, U5.2
- net BP8.OUT2: now reaches JPP2.41, JPP2.42
- net BP8.OUT2: now also R42.2, U5.6
- net BP9.OUT2: now reaches JPP2.46, JPP2.47
- net BP9.OUT2: now also R47.2, U4.6
- net BP1.OUT2: now reaches JPP2.6, JPP2.7
- net BP1.OUT2: now also R5.2, U2.6
- net NI1: now reaches J1.1
- net NI1: now also U1.2
- net NI2: now reaches J1.2
- net NI2: now also U1.6
- net NI3: now reaches J1.3
- net NI3: now also U3.6
- net NI4: now reaches J1.4
- net NI4: now also U3.9
- net NI5: now reaches J1.5
- net NI5: now also U1.9, U4.2
- net NI6: now reaches J1.6
- net NI6: now also U1.13
- net NI7: now reaches J1.7
- net NI7: now also U3.13
- net NI8: now reaches J1.8
- net NI9: now reaches J1.9
- net NI9: now also U2.2
- net OR8: now reaches J2.10 (Pin_10)
- net OR8: now also U5.4
- net OR9: now reaches J2.11 (Pin_11)
- net OR9: now also U4.4
- net OR1: now reaches J2.3 (Pin_3)
- net OR1: now also U2.4
- net OR2: now reaches J2.4 (Pin_4)
- net OR2: now also U2.10
- net OR3: now reaches J2.5 (Pin_5)
- net OR3: now also U4.10
- net OR4: now reaches J2.6 (Pin_6)
- net OR4: now also U4.11
- net OR5: now reaches J2.7 (Pin_7)
- net OR5: now also U2.11
- net OR6: now reaches J2.8 (Pin_8)
- net OR6: now also U3.3
- net OR7: now reaches J2.9 (Pin_9)
- net OR7: now also U5.3
- new net AND1: U1.3, U2.5
- new net AND2: U1.4, U2.8
- new net AND3: U3.4, U4.8
- new net AND4: U3.10, U4.12
- new net AND5: U1.10, U2.12
- new net AND6: U1.11, U3.1
- new net AND7: U3.11, U5.1
- new net AND8: U4.3, U5.5
- new net AND9: U2.3, U4.5
Other:
- note added: "Porte logique AND 1\n"
- note added: "Porte logique AND 2\n\n"
- note added: "Porte logique AND 3\n\n"
- note added: "Porte logique OR 1\n\n"
- note added: "Porte logique OR 2\n\n"
- note added: "Porte logique OR 3\n\n"
- moved on the sheet: J1, J2, JPP1, JPP2, R12, R6
